File: UnifiedMotherboard.kicad_sch (KiCad schematic)
At the start: 46 parts, among them J1 USB_C_Receptacle_USB2.0, J2 Conn_2Rows-75Pins, SW1 SW_Push_45deg, SW2 SW_Push_45deg, SW3 SW_PUSH, U1 RP2040, U2 W25Q128JVS, U3 USBLC6-2SC6, U4 XC6206PxxxMR, U5 ATMEGA32U2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

Commit message: Updated schematic and pcb layout
Parts:
- removed J2: Conn_2Rows-75Pins, symbol Connector_Generic:Conn_2Rows-75Pins
- added U6: ~, symbol unified_motherboard:unified_motherboard
Connections:
- new net: U6.10 (GND), U6.13 (GND), U6.16 (GND), U6.22 (GND)
